Commit message: update

File: urdf/blueboat_enu_sim.xacro (robot description, xacro)
@@ -51,5 +51,5 @@
       <parent link="${prefix}base_link"/>
       <child link="${prefix}lidar_front"/>
-      <origin xyz="0.115 -0.36 -1.25" rpy="3.1416 0.0 0.0"/>
+      <origin xyz="0.115 -0.36 -0.25" rpy="3.1416 0.0 0.0"/>
     </joint>
     <!-- GPS -->

Commit message: Rotate lidar +90 to simulate the real blueboat setup

File: urdf/blueboat_enu_sim.xacro (robot description, xacro)
@@ -51,5 +51,5 @@
       <parent link="${prefix}base_link"/>
       <child link="${prefix}lidar_front"/>
-      <origin xyz="0.115 -0.36 -0.25" rpy="3.1416 0.0 0.0"/>
+      <origin xyz="0.39 -0.36 -0.25" rpy="3.1416 0.0 1.5708"/>
     </joint>
     <!-- GPS -->
@@ -65,5 +65,5 @@
       <parent link="${prefix}base_link"/>
       <child link="${prefix}imu_link"/>
-      <origin xyz="0.35 -0.35 -0.2" rpy="0.0 0.0 0.0"/>
+      <origin xyz="0.39 -0.36 -0.25" rpy="3.1416 0.0 1.5708"/>
     </joint>
     <!-- =========================================================
