Commit message: Fixing name problems

File: urdf/blueboat.xacro (robot description, xacro)
@@ -8,5 +8,5 @@
         <origin rpy="3.1416 0 -1.5708" xyz="0 0 0" />
         <geometry>
-          <mesh filename="package://blueboat_description/meshes/blueboat.dae" scale="1 1 1"/>
+          <mesh filename="package://blueboat_cirtesu_description/meshes/blueboat.dae" scale="1 1 1"/>
         </geometry>
         <material name="blue">
@@ -17,5 +17,5 @@
         <origin rpy="3.1416 0 -1.5708" xyz="0 0 0" />
         <geometry>
-          <mesh filename="package://blueboat_description/meshes/blueboat.dae" scale="1 1 1"/>
+          <mesh filename="package://blueboat_cirtesu_description/meshes/blueboat.dae" scale="1 1 1"/>
         </geometry>
       </collision>
@@ -59,4 +59,4 @@
   </xacro:macro>
   <!-- LLAMAR A LA MACRO -->
-  <xacro:blueboat_macro prefix="blueboat_"/>
+  <xacro:blueboat_macro prefix="blueboat/"/>
 </robot>

File: urdf/blueboat_enu.xacro (robot description, xacro)
@@ -19,5 +19,5 @@
         <origin rpy="3.1416 0 -1.5708" xyz="0 0 0"/>
         <geometry>
-          <mesh filename="package://blueboat_description/meshes/blueboat.dae" scale="1 1 1"/>
+          <mesh filename="package://blueboat_cirtesu_description/meshes/blueboat.dae" scale="1 1 1"/>
         </geometry>
         <material name="blue">
@@ -28,5 +28,5 @@
         <origin rpy="3.1416 0 -1.5708" xyz="0 0 0"/>
         <geometry>
-          <mesh filename="package://blueboat_description/meshes/blueboat.dae" scale="1 1 1"/>
+          <mesh filename="package://blueboat_cirtesu_description/meshes/blueboat.dae" scale="1 1 1"/>
         </geometry>
       </collision>

Commit message: xyz propellers

File: urdf/blueboat.xacro (robot description, xacro)
@@ -11,5 +11,5 @@
       <parent link="${prefix}base_link"/>
       <child link="${prefix}left_thruster_link"/>
-      <origin xyz="-0.472 -0.3 0.0245" rpy="1.57 0.0 0.0"/>
+      <origin xyz="-0.1908 -0.294712 0.284077" rpy="0.0 0.0 0.0"/>
     </joint>
     <!-- Thruster derecho -->
@@ -18,5 +18,5 @@
       <parent link="${prefix}base_link"/>
       <child link="${prefix}right_thruster_link"/>
-      <origin xyz="-0.472 0.26 0.0245" rpy="1.57 0.0 0.0"/>
+      <origin xyz="-0.190825 0.259452 0.284077" rpy="0.0 0.0 0.0"/>
     </joint>
   </xacro:macro>

Commit message: Remove blueboat/ in joint name

File: urdf/blueboat.xacro (robot description, xacro)
@@ -28,9 +28,9 @@
       <param name="lookup_csv">$(arg lookup_csv)</param>
     </hardware>
-    <joint name="blueboat/left_thruster_joint">
+    <joint name="left_thruster_joint">
       <command_interface name="effort"/>
       <state_interface name="effort"/>
     </joint>
-    <joint name="blueboat/right_thruster_joint">
+    <joint name="right_thruster_joint">
       <command_interface name="effort"/>
       <state_interface name="effort"/>

Commit message: blueboat

File: urdf/blueboat.xacro (robot description, xacro)
@@ -28,9 +28,9 @@
       <param name="lookup_csv">$(arg lookup_csv)</param>
     </hardware>
-    <joint name="left_thruster_joint">
+    <joint name="blueboat/left_thruster_joint">
       <command_interface name="effort"/>
       <state_interface name="effort"/>
     </joint>
-    <joint name="right_thruster_joint">
+    <joint name="blueboat/right_thruster_joint">
       <command_interface name="effort"/>
       <state_interface name="effort"/>

Commit message: invert yaw 180

File: urdf/blueboat.xacro (robot description, xacro)
@@ -1,6 +1,8 @@
 <?xml version="1.0"?>
 <robot xmlns:xacro="http://www.ros.org/wiki/xacro" name="blueboat">
-  <xacro:arg name="environment" default="sim"/>
+  <xacro:arg name="environment" default="real"/>
   <xacro:arg name="lookup_csv" default=""/>
+  <xacro:arg name="pwm_channels" default="0,2"/>
+  <xacro:arg name="stonefish_topic" default="/catamaran/controller/thruster_setpoints_sim"/>
   <xacro:macro name="blueboat_thrusters_macro" params="prefix">
     <!-- Link base mínimo -->
@@ -11,5 +13,5 @@
       <parent link="${prefix}base_link"/>
       <child link="${prefix}left_thruster_link"/>
-      <origin xyz="-0.1908 -0.294712 0.284077" rpy="0.0 0.0 0.0"/>
+      <origin xyz="-0.472 -0.3 0.0245" rpy="0.0 0.0 3.14159265"/>
     </joint>
     <!-- Thruster derecho -->
@@ -18,5 +20,5 @@
       <parent link="${prefix}base_link"/>
       <child link="${prefix}right_thruster_link"/>
-      <origin xyz="-0.190825 0.259452 0.284077" rpy="0.0 0.0 0.0"/>
+      <origin xyz="-0.472 0.3 0.0245" rpy="0.0 0.0 3.14159265"/>
     </joint>
   </xacro:macro>
@@ -27,12 +29,16 @@
       <param name="environment">$(arg environment)</param>
       <param name="lookup_csv">$(arg lookup_csv)</param>
+      <param name="pwm_channels">$(arg pwm_channels)</param>
+      <param name="stonefish_topic">$(arg stonefish_topic)</param>
     </hardware>
     <joint name="blueboat/left_thruster_joint">
       <command_interface name="effort"/>
       <state_interface name="effort"/>
+      <param name="inverted">false</param>
     </joint>
     <joint name="blueboat/right_thruster_joint">
       <command_interface name="effort"/>
       <state_interface name="effort"/>
+      <param name="inverted">true</param>
     </joint>
   </ros2_control>

Commit message: sura sensors system

File: urdf/blueboat.xacro (robot description, xacro)
@@ -6,7 +6,5 @@
   <xacro:arg name="stonefish_topic" default="/catamaran/controller/thruster_setpoints_sim"/>
   <xacro:macro name="blueboat_thrusters_macro" params="prefix">
-    <!-- Link base mínimo -->
     <link name="${prefix}base_link"/>
-    <!-- Thruster izquierdo -->
     <link name="${prefix}left_thruster_link"/>
     <joint name="${prefix}left_thruster_joint" type="fixed">
@@ -15,5 +13,4 @@
       <origin xyz="-0.472 -0.3 0.0245" rpy="0.0 0.0 3.14159265"/>
     </joint>
-    <!-- Thruster derecho -->
     <link name="${prefix}right_thruster_link"/>
     <joint name="${prefix}right_thruster_joint" type="fixed">
@@ -22,9 +19,15 @@
       <origin xyz="-0.472 0.3 0.0245" rpy="0.0 0.0 3.14159265"/>
     </joint>
+    <link name="${prefix}imu_link"/>
+    <joint name="${prefix}imu_joint" type="fixed">
+      <parent link="${prefix}base_link"/>
+      <child link="${prefix}imu_link"/>
+      <origin xyz="0 0 0" rpy="0 0 0"/>
+    </joint>
   </xacro:macro>
   <xacro:blueboat_thrusters_macro prefix="blueboat/"/>
   <ros2_control name="ThrustersSystem" type="system">
     <hardware>
-      <plugin>thrusters_hardware_interface/ThrustersSystem</plugin>
+      <plugin>sura_hardware_interface/ThrustersSystem</plugin>
       <param name="environment">$(arg environment)</param>
       <param name="lookup_csv">$(arg lookup_csv)</param>
@@ -43,3 +46,20 @@
     </joint>
   </ros2_control>
+  <ros2_control name="SensorsSystem" type="system">
+    <hardware>
+      <plugin>sura_hardware_interface/SensorsSystem</plugin>
+    </hardware>
+    <sensor name="imu_sensor">
+      <state_interface name="orientation.x"/>
+      <state_interface name="orientation.y"/>
+      <state_interface name="orientation.z"/>
+      <state_interface name="orientation.w"/>
+      <state_interface name="angular_velocity.x"/>
+      <state_interface name="angular_velocity.y"/>
+      <state_interface name="angular_velocity.z"/>
+      <state_interface name="linear_acceleration.x"/>
+      <state_interface name="linear_acceleration.y"/>
+      <state_interface name="linear_acceleration.z"/>
+    </sensor>
+  </ros2_control>
 </robot>

Commit message: Update blueboat xacro files

File: urdf/blueboat.xacro (robot description, xacro)
@@ -5,5 +5,8 @@
   <xacro:arg name="pwm_channels" default="0,2"/>
   <xacro:arg name="stonefish_topic" default="/catamaran/controller/thruster_setpoints_sim"/>
-  <xacro:macro name="blueboat_thrusters_macro" params="prefix">
+  <xacro:macro name="blueboat_thrusters_macro" params="prefix environment">
+    <xacro:property name="thruster_yaw" value="${0.0 if environment == 'sim' else 3.14159265}"/>
+    <xacro:property name="left_thruster_y" value="${-0.28 if environment == 'sim' else -0.3}"/>
+    <xacro:property name="right_thruster_y" value="${0.28 if environment == 'sim' else 0.3}"/>
     <link name="${prefix}base_link"/>
     <link name="${prefix}left_thruster_link"/>
@@ -11,5 +14,5 @@
       <parent link="${prefix}base_link"/>
       <child link="${prefix}left_thruster_link"/>
-      <origin xyz="-0.472 -0.3 0.0245" rpy="0.0 0.0 3.14159265"/>
+      <origin xyz="-0.472 ${left_thruster_y} 0.0245" rpy="0.0 0.0 ${thruster_yaw}"/>
     </joint>
     <link name="${prefix}right_thruster_link"/>
@@ -17,5 +20,5 @@
       <parent link="${prefix}base_link"/>
       <child link="${prefix}right_thruster_link"/>
-      <origin xyz="-0.472 0.3 0.0245" rpy="0.0 0.0 3.14159265"/>
+      <origin xyz="-0.472 ${right_thruster_y} 0.0245" rpy="0.0 0.0 ${thruster_yaw}"/>
     </joint>
     <link name="${prefix}imu_link"/>
@@ -26,5 +29,5 @@
     </joint>
   </xacro:macro>
-  <xacro:blueboat_thrusters_macro prefix="blueboat/"/>
+  <xacro:blueboat_thrusters_macro prefix="blueboat/" environment="$(arg environment)"/>
   <ros2_control name="ThrustersSystem" type="system">
     <hardware>

File: urdf/blueboat_enu_sim.xacro (robot description, xacro)
@@ -73,6 +73,6 @@
          ========================================================= -->
     <!-- En tu escena Stonefish:
-         Thruster_R -> xyz="-0.472 0.26 0.0245" rpy="1.57 0 0"
-         Thruster_L -> xyz="-0.472 -0.3 0.0245" rpy="1.57 0 0"
+         Thruster_R -> xyz="-0.472 0.28 0.0245" rpy="1.57 0 0"
+         Thruster_L -> xyz="-0.472 -0.28 0.0245" rpy="1.57 0 0"
     -->
     <link name="${prefix}left_thruster_link"/>
@@ -80,5 +80,5 @@
       <parent link="${prefix}base_link"/>
       <child link="${prefix}left_thruster_link"/>
-      <origin xyz="-0.472 -0.3 0.0245" rpy="1.57 0.0 0.0"/>
+      <origin xyz="-0.472 -0.28 0.0245" rpy="0.0 0.0 0.0"/>
     </joint>
     <link name="${prefix}right_thruster_link"/>
@@ -86,5 +86,5 @@
       <parent link="${prefix}base_link"/>
       <child link="${prefix}right_thruster_link"/>
-      <origin xyz="-0.472 0.26 0.0245" rpy="1.57 0.0 0.0"/>
+      <origin xyz="-0.472 0.28 0.0245" rpy="0.0 0.0 0.0"/>
     </joint>
   </xacro:macro>

Commit message: update xacro

File: urdf/blueboat.xacro (robot description, xacro)
@@ -5,4 +5,7 @@
   <xacro:arg name="pwm_channels" default="0,2"/>
   <xacro:arg name="stonefish_topic" default="/catamaran/controller/thruster_setpoints_sim"/>
+  <xacro:arg name="gps_protocol" default="ubx"/>
+  <xacro:arg name="gps_serial_port" default="/dev/ttyAMA5"/>
+  <xacro:arg name="gps_baudrate" default="230400"/>
   <xacro:macro name="blueboat_thrusters_macro" params="prefix environment">
     <xacro:property name="thruster_yaw" value="${0.0 if environment == 'sim' else 3.14159265}"/>
@@ -27,4 +30,10 @@
       <child link="${prefix}imu_link"/>
       <origin xyz="0 0 0" rpy="0 0 0"/>
+    </joint>
+    <link name="gps_frame"/>
+    <joint name="${prefix}gps_joint" type="fixed">
+      <parent link="${prefix}base_link"/>
+      <child link="gps_frame"/>
+      <origin xyz="0.39 -0.36 -0.05" rpy="3.1416 0 1.57"/>
     </joint>
   </xacro:macro>
@@ -52,4 +61,8 @@
     <hardware>
       <plugin>sura_hardware_interface/SensorsSystem</plugin>
+      <param name="environment">$(arg environment)</param>
+      <param name="gps_protocol">$(arg gps_protocol)</param>
+      <param name="gps_serial_port">$(arg gps_serial_port)</param>
+      <param name="gps_baudrate">$(arg gps_baudrate)</param>
     </hardware>
     <sensor name="imu_sensor">
@@ -75,4 +88,10 @@
       <state_interface name="present"/>
     </sensor>
+    <sensor name="gps_sensor">
+      <state_interface name="gps.latitude"/>
+      <state_interface name="gps.longitude"/>
+      <state_interface name="gps.altitude"/>
+      <state_interface name="gps.valid"/>
+    </sensor>
   </ros2_control>
 </robot>

Commit message: Add ActuatorSystem

File: urdf/blueboat.xacro (robot description, xacro)
@@ -4,4 +4,5 @@
   <xacro:arg name="lookup_csv" default=""/>
   <xacro:arg name="pwm_channels" default="0,2"/>
+  <xacro:arg name="status_light_channel" default="1"/>
   <xacro:arg name="stonefish_topic" default="/catamaran/controller/thruster_setpoints_sim"/>
   <xacro:arg name="gps_protocol" default="ubx"/>
@@ -37,4 +38,10 @@
       <origin xyz="0.39 -0.36 -0.05" rpy="3.1416 0 1.57"/>
     </joint>
+    <link name="${prefix}status_light_link"/>
+    <joint name="${prefix}status_light_joint" type="fixed">
+      <parent link="${prefix}base_link"/>
+      <child link="${prefix}status_light_link"/>
+      <origin xyz="0 0 0" rpy="0 0 0"/>
+    </joint>
   </xacro:macro>
   <xacro:blueboat_thrusters_macro prefix="blueboat/" environment="$(arg environment)"/>
@@ -56,4 +63,15 @@
       <state_interface name="effort"/>
       <param name="inverted">true</param>
+    </joint>
+  </ros2_control>
+  <ros2_control name="ActuatorsSystem" type="system">
+    <hardware>
+      <plugin>sura_hardware_interface/ActuatorsSystem</plugin>
+      <param name="environment">$(arg environment)</param>
+      <param name="status_light_channel">$(arg status_light_channel)</param>
+    </hardware>
+    <joint name="blueboat/status_light_joint">
+      <command_interface name="enabled"/>
+      <state_interface name="enabled"/>
     </joint>
   </ros2_control>

Commit message: First functional seaport demo

File: urdf/blueboat.xacro (robot description, xacro)
@@ -5,8 +5,10 @@
   <xacro:arg name="pwm_channels" default="0,2"/>
   <xacro:arg name="status_light_channel" default="1"/>
+  <xacro:arg name="enable_status_light" default="true"/>
   <xacro:arg name="stonefish_topic" default="/catamaran/controller/thruster_setpoints_sim"/>
   <xacro:arg name="gps_protocol" default="ubx"/>
   <xacro:arg name="gps_serial_port" default="/dev/ttyAMA5"/>
   <xacro:arg name="gps_baudrate" default="230400"/>
+  <xacro:arg name="enable_battery" default="true"/>
   <xacro:macro name="blueboat_thrusters_macro" params="prefix environment">
     <xacro:property name="thruster_yaw" value="${0.0 if environment == 'sim' else 3.14159265}"/>
@@ -65,15 +67,17 @@
     </joint>
   </ros2_control>
-  <ros2_control name="ActuatorsSystem" type="system">
-    <hardware>
-      <plugin>sura_hardware_interface/ActuatorsSystem</plugin>
-      <param name="environment">$(arg environment)</param>
-      <param name="status_light_channel">$(arg status_light_channel)</param>
-    </hardware>
-    <joint name="blueboat/status_light_joint">
-      <command_interface name="enabled"/>
-      <state_interface name="enabled"/>
-    </joint>
-  </ros2_control>
+  <xacro:if value="$(arg enable_status_light)">
+    <ros2_control name="ActuatorsSystem" type="system">
+      <hardware>
+        <plugin>sura_hardware_interface/ActuatorsSystem</plugin>
+        <param name="environment">$(arg environment)</param>
+        <param name="status_light_channel">$(arg status_light_channel)</param>
+      </hardware>
+      <joint name="blueboat/status_light_joint">
+        <command_interface name="enabled"/>
+        <state_interface name="enabled"/>
+      </joint>
+    </ros2_control>
+  </xacro:if>
   <ros2_control name="SensorsSystem" type="system">
     <hardware>
@@ -101,9 +105,11 @@
       <state_interface name="magnetic_field.z"/>
     </sensor>
-    <sensor name="battery_sensor">
-      <state_interface name="voltage"/>
-      <state_interface name="current"/>
-      <state_interface name="present"/>
-    </sensor>
+    <xacro:if value="$(arg enable_battery)">
+      <sensor name="battery_sensor">
+        <state_interface name="voltage"/>
+        <state_interface name="current"/>
+        <state_interface name="present"/>
+      </sensor>
+    </xacro:if>
     <sensor name="gps_sensor">
       <state_interface name="gps.latitude"/>
