Commit message: Ros control adaptation

File: urdf/blueboat_enu_real.xacro (robot description, xacro)
@@ -1,4 +1,6 @@
 <?xml version="1.0"?>
 <robot xmlns:xacro="http://www.ros.org/wiki/xacro" name="blueboat">
+  <xacro:arg name="environment" default="real"/>
+  <xacro:arg name="lookup_csv" default=""/>
   <xacro:macro name="blueboat_macro" params="prefix">
     <!-- =========================================================
@@ -65,4 +67,16 @@
       <origin xyz="0.39 -0.36 -0.05" rpy="3.1416 0 1.57"/>
     </joint>
+  <link name="${prefix}left_thruster_link"/>
+  <joint name="${prefix}left_thruster_joint" type="fixed">
+    <parent link="${prefix}base_link"/>
+    <child link="${prefix}left_thruster_link"/>
+    <origin xyz="X_LEFT Y_LEFT Z_LEFT" rpy="0 0 0"/>
+  </joint>
+  <link name="${prefix}right_thruster_link"/>
+  <joint name="${prefix}right_thruster_joint" type="fixed">
+    <parent link="${prefix}base_link"/>
+    <child link="${prefix}right_thruster_link"/>
+    <origin xyz="X_RIGHT Y_RIGHT Z_RIGHT" rpy="0 0 0"/>
+  </joint>
   </xacro:macro>
   <xacro:blueboat_macro prefix="blueboat/"/>

Commit message: Rename BlueBoat description package

File: urdf/blueboat_enu_real.xacro (robot description, xacro)
@@ -21,5 +21,5 @@
         <origin rpy="3.1416 0 -1.5708" xyz="0 0 0"/>
         <geometry>
-          <mesh filename="package://blueboat_cirtesu_description/meshes/blueboat.dae" scale="1 1 1"/>
+          <mesh filename="package://blueboat_description/meshes/blueboat.dae" scale="1 1 1"/>
         </geometry>
         <material name="blue">
@@ -30,5 +30,5 @@
         <origin rpy="3.1416 0 -1.5708" xyz="0 0 0"/>
         <geometry>
-          <mesh filename="package://blueboat_cirtesu_description/meshes/blueboat.dae" scale="1 1 1"/>
+          <mesh filename="package://blueboat_description/meshes/blueboat.dae" scale="1 1 1"/>
         </geometry>
       </collision>
