Commit message: Update BlueBoat description and ros2_control config

File: urdf/blueboat.urdf.xacro (robot description, xacro)
@@ -1,22 +1,11 @@
 <?xml version="1.0"?>
-<robot xmlns:xacro="http://www.ros.org/wiki/xacro" name="blueboat">
+<robot xmlns:xacro="http://www.ros.org/wiki/xacro" name="blueboat" family="$(arg family)">
   <xacro:arg name="environment" default="real"/>
   <xacro:arg name="robot_namespace" default="blueboat"/>
-  <xacro:arg name="lookup_csv" default=""/>
-  <xacro:arg name="pwm_channels" default="0,2"/>
-  <xacro:arg name="status_light_channel" default="1"/>
-  <xacro:arg name="stonefish_topic" default="/blueboat/catamaran/controller/thruster_setpoints_sim"/>
-  <xacro:arg name="gps_protocol" default="ubx"/>
-  <xacro:arg name="gps_serial_port" default="/dev/ttyAMA5"/>
-  <xacro:arg name="gps_baudrate" default="230400"/>
+  <xacro:arg name="family" default="surface"/>
+  <xacro:arg name="lookup_csv" default="config/m200_lookup.csv"/>
+  <xacro:arg name="stonefish_topic" default="/$(arg robot_namespace)/controller/thruster_setpoints_sim"/>
   <xacro:property name="robot_prefix" value="$(arg robot_namespace)/"/>
-  <xacro:property name="robot_namespace" value="$(arg robot_namespace)"/>
-  <xacro:property name="environment" value="$(arg environment)"/>
-  <xacro:property name="thruster_yaw" value="${0.0 if environment == 'sim' else 3.14159265}"/>
-  <xacro:property name="left_thruster_y" value="${-0.28 if environment == 'sim' else -0.3}"/>
-  <xacro:property name="right_thruster_y" value="${0.28 if environment == 'sim' else 0.3}"/>
-  <!-- ========================================================= -->
   <!-- TF -->
-  <!-- ========================================================= -->
   <link name="${robot_prefix}base_link_enu" tf_type="base"/>
   <link name="${robot_prefix}base_link" tf_type="base"/>
@@ -26,7 +15,5 @@
     <origin xyz="0 0 0" rpy="3.14159265359 0 0"/>
   </joint>
-  <!-- ========================================================= -->
   <!-- Sensors -->
-  <!-- ========================================================= -->
   <link name="${robot_prefix}imu_link" tf_type="sensor"/>
   <joint name="${robot_prefix}imu_joint" type="fixed">
@@ -47,12 +34,16 @@
     <origin xyz="0.39 -0.36 -0.05" rpy="3.1416 0 1.57"/>
   </joint>
-  <!-- ========================================================= -->
+  <link name="${robot_prefix}altimeter_link" tf_type="sensor"/>
+  <joint name="${robot_prefix}altimeter_joint" type="fixed">
+    <parent link="${robot_prefix}base_link"/>
+    <child link="${robot_prefix}altimeter_link"/>
+    <origin xyz="-0.240439 0.067376 -0.35413" rpy="3.1416 0 1.57"/>
+  </joint>
   <!-- Thrusters -->
-  <!-- ========================================================= -->
   <link name="${robot_prefix}left_thruster_link" tf_type="thruster"/>
   <joint name="${robot_prefix}left_thruster_joint" type="fixed">
     <parent link="${robot_prefix}base_link"/>
     <child link="${robot_prefix}left_thruster_link"/>
-    <origin xyz="-0.472 ${left_thruster_y} 0.0245" rpy="0.0 0.0 ${thruster_yaw}"/>
+    <origin xyz="-0.472 -0.28 0.0245" rpy="0.0 0.0 0.0"/>
   </joint>
   <link name="${robot_prefix}right_thruster_link" tf_type="thruster"/>
@@ -60,9 +51,7 @@
     <parent link="${robot_prefix}base_link"/>
     <child link="${robot_prefix}right_thruster_link"/>
-    <origin xyz="-0.472 ${right_thruster_y} 0.0245" rpy="0.0 0.0 ${thruster_yaw}"/>
+    <origin xyz="-0.472 0.28 0.0245" rpy="0.0 0.0 0.0"/>
   </joint>
-  <!-- ========================================================= -->
   <!-- Actuators -->
-  <!-- ========================================================= -->
   <!--
   <link name="${robot_prefix}status_light_link" tf_type="actuator"/>
@@ -73,53 +62,31 @@
   </joint>
   -->
-  <!-- ========================================================= -->
   <!-- ROS2 CONTROL -->
-  <!-- ========================================================= -->
-  <ros2_control name="ThrustersSystem" type="system">
+  <ros2_control name="blueboat_thrusters" type="system">
     <hardware>
       <plugin>sura_hardware_interface/ThrustersSystem</plugin>
       <param name="environment">$(arg environment)</param>
-      <param name="lookup_csv">$(arg lookup_csv)</param>
-      <param name="pwm_channels">$(arg pwm_channels)</param>
-      <param name="stonefish_topic">$(arg stonefish_topic)</param>
     </hardware>
     <joint name="${robot_prefix}left_thruster_joint">
       <command_interface name="effort"/>
       <state_interface name="effort"/>
-      <param name="role">thruster</param>
-      <param name="controller">body_force_controller</param>
+      <param name="lookup_csv">$(arg lookup_csv)</param>
+      <param name="stonefish_topic">$(arg stonefish_topic)</param>
       <param name="inverted">false</param>
+      <param name="channel">0</param>
     </joint>
     <joint name="${robot_prefix}right_thruster_joint">
       <command_interface name="effort"/>
       <state_interface name="effort"/>
-      <param name="role">thruster</param>
-      <param name="controller">body_force_controller</param>
+      <param name="lookup_csv">$(arg lookup_csv)</param>
+      <param name="stonefish_topic">$(arg stonefish_topic)</param>
       <param name="inverted">true</param>
+      <param name="channel">2</param>
     </joint>
   </ros2_control>
-  <!--
-  <ros2_control name="ActuatorsSystem" type="system">
-    <hardware>
-      <plugin>sura_hardware_interface/ActuatorsSystem</plugin>
-      <param name="environment">$(arg environment)</param>
-      <param name="status_light_channel">1</param>
-    </hardware>
-    <joint name="${robot_prefix}status_light_joint">
-      <command_interface name="enabled"/>
-      <state_interface name="enabled"/>
-      <param name="role">actuator</param>
-      <param name="controller">status_light_controller</param>
-    </joint>
-  </ros2_control>
-  -->
-  <ros2_control name="SensorsSystem" type="system">
+  <ros2_control name="blueboat_sensors" type="system">
     <hardware>
       <plugin>sura_hardware_interface/SensorsSystem</plugin>
       <param name="environment">$(arg environment)</param>
-      <param name="robot_namespace">$(arg robot_namespace)</param>
-      <param name="gps_protocol">$(arg gps_protocol)</param>
-      <param name="gps_serial_port">$(arg gps_serial_port)</param>
-      <param name="gps_baudrate">$(arg gps_baudrate)</param>
     </hardware>
     <sensor name="imu_sensor">
@@ -128,5 +95,6 @@
       <param name="read_rate_hz">200.0</param>
       <param name="frame_id">${robot_prefix}imu_link</param>
-      <param name="stonefish_topic">/${robot_namespace}/stonefish/sensors/imu</param>
+      <param name="stonefish_topic">/$(arg robot_namespace)/stonefish/sensors/imu</param>
+      <param name="msg_type">sensor_msgs/msg/Imu</param>
       <state_interface name="orientation.x"/>
       <state_interface name="orientation.y"/>
@@ -145,10 +113,10 @@
       <param name="read_rate_hz">50.0</param>
       <param name="frame_id">${robot_prefix}imu_link</param>
-      <param name="stonefish_topic">/${robot_namespace}/stonefish/sensors/magnetometer</param>
+      <param name="stonefish_topic">/$(arg robot_namespace)/stonefish/sensors/magnetometer</param>
+      <param name="msg_type">sensor_msgs/msg/MagneticField</param>
       <state_interface name="magnetic_field.x"/>
       <state_interface name="magnetic_field.y"/>
       <state_interface name="magnetic_field.z"/>
     </sensor>
-    <!--
     <sensor name="battery_sensor">
       <param name="interface">sura_hardware_interface/BatteryInterface</param>
@@ -160,11 +128,23 @@
       <state_interface name="present"/>
     </sensor>
-    -->
+    <sensor name="altimeter_sensor">
+      <param name="interface">sura_hardware_interface/AltimeterBlueboatInterface</param>
+      <param name="broadcaster">altimeter_broadcaster</param>
+      <param name="read_rate_hz">20.0</param>
+      <param name="serial_port">/dev/ttyAMA3</param>
+      <param name="baudrate">115200</param>
+      <param name="frame_id">${robot_prefix}altimeter_link</param>
+      <state_interface name="altitude"/>
+    </sensor>
     <sensor name="gps_sensor">
       <param name="interface">sura_hardware_interface/GpsInterface</param>
       <param name="broadcaster">gps_broadcaster</param>
       <param name="read_rate_hz">1.0</param>
+      <param name="gps_protocol">ubx</param>
+      <param name="gps_serial_port">/dev/ttyAMA5</param>
+      <param name="gps_baudrate">230400</param>
       <param name="frame_id">${robot_prefix}gps_frame</param>
-      <param name="stonefish_topic">/${robot_namespace}/stonefish/sensors/gps</param>
+      <param name="stonefish_topic">/$(arg robot_namespace)/stonefish/sensors/gps</param>
+      <param name="msg_type">sensor_msgs/msg/NavSatFix</param>
       <state_interface name="gps.latitude"/>
       <state_interface name="gps.longitude"/>
@@ -173,3 +153,17 @@
     </sensor>
   </ros2_control>
+  <ros2_control name="blueboat_actuators" type="system">
+    <hardware>
+      <plugin>sura_hardware_interface/ActuatorsSystem</plugin>
+      <param name="environment">$(arg environment)</param>
+      <param name="status_light_channel">1</param>
+    </hardware>
+    <joint name="${robot_prefix}status_light_joint">
+      <param name="interface">sura_hardware_interface/LightBlueboatInterface</param>
+      <command_interface name="enabled"/>
+      <state_interface name="enabled"/>
+      <param name="channel">1</param>
+      <param name="controller">status_light_controller</param>
+    </joint>
+  </ros2_control>
 </robot>

Commit message: integration

File: urdf/blueboat.urdf.xacro (robot description, xacro)
@@ -1,85 +1,81 @@
 <?xml version="1.0"?>
-<robot xmlns:xacro="http://www.ros.org/wiki/xacro" name="blueboat" family="$(arg family)">
+<robot xmlns:xacro="http://www.ros.org/wiki/xacro" name="blueboat" family="surface">
+  <xacro:arg name="robot_name" default="blueboat"/>
   <xacro:arg name="environment" default="real"/>
-  <xacro:arg name="robot_namespace" default="blueboat"/>
-  <xacro:arg name="family" default="surface"/>
-  <xacro:arg name="lookup_csv" default="config/m200_lookup.csv"/>
-  <xacro:arg name="stonefish_topic" default="/$(arg robot_namespace)/controller/thruster_setpoints_sim"/>
-  <xacro:property name="robot_prefix" value="$(arg robot_namespace)/"/>
   <!-- TF -->
-  <link name="${robot_prefix}base_link_enu" tf_type="base"/>
-  <link name="${robot_prefix}base_link" tf_type="base"/>
-  <joint name="${robot_prefix}enu_to_ned_joint" type="fixed">
-    <parent link="${robot_prefix}base_link_enu"/>
-    <child link="${robot_prefix}base_link"/>
+  <link name="$(arg robot_name)/base_link_enu" tf_type="base"/>
+  <link name="$(arg robot_name)/base_link" tf_type="base"/>
+  <joint name="$(arg robot_name)/enu_to_ned_joint" type="fixed">
+    <parent link="$(arg robot_name)/base_link_enu"/>
+    <child link="$(arg robot_name)/base_link"/>
     <origin xyz="0 0 0" rpy="3.14159265359 0 0"/>
   </joint>
   <!-- Sensors -->
-  <link name="${robot_prefix}imu_link" tf_type="sensor"/>
-  <joint name="${robot_prefix}imu_joint" type="fixed">
-    <parent link="${robot_prefix}base_link"/>
-    <child link="${robot_prefix}imu_link"/>
+  <link name="$(arg robot_name)/imu_link" tf_type="sensor"/>
+  <joint name="$(arg robot_name)/imu_joint" type="fixed">
+    <parent link="$(arg robot_name)/base_link"/>
+    <child link="$(arg robot_name)/imu_link"/>
     <origin xyz="0 0 0" rpy="0 0 0"/>
   </joint>
-  <link name="${robot_prefix}lidar_front" tf_type="sensor"/>
-  <joint name="${robot_prefix}lidar_joint" type="fixed">
-    <parent link="${robot_prefix}base_link"/>
-    <child link="${robot_prefix}lidar_front"/>
+  <link name="$(arg robot_name)/lidar_front" tf_type="sensor"/>
+  <joint name="$(arg robot_name)/lidar_joint" type="fixed">
+    <parent link="$(arg robot_name)/base_link"/>
+    <child link="$(arg robot_name)/lidar_front"/>
     <origin xyz="0.39 -0.36 -0.05" rpy="3.1416 0 1.57"/>
   </joint>
-  <link name="${robot_prefix}gps_frame" tf_type="sensor"/>
-  <joint name="${robot_prefix}gps_joint" type="fixed">
-    <parent link="${robot_prefix}base_link"/>
-    <child link="${robot_prefix}gps_frame"/>
+  <link name="$(arg robot_name)/gps_frame" tf_type="sensor"/>
+  <joint name="$(arg robot_name)/gps_joint" type="fixed">
+    <parent link="$(arg robot_name)/base_link"/>
+    <child link="$(arg robot_name)/gps_frame"/>
     <origin xyz="0.39 -0.36 -0.05" rpy="3.1416 0 1.57"/>
   </joint>
-  <link name="${robot_prefix}altimeter_link" tf_type="sensor"/>
-  <joint name="${robot_prefix}altimeter_joint" type="fixed">
-    <parent link="${robot_prefix}base_link"/>
-    <child link="${robot_prefix}altimeter_link"/>
+  <link name="$(arg robot_name)/altimeter_link" tf_type="sensor"/>
+  <joint name="$(arg robot_name)/altimeter_joint" type="fixed">
+    <parent link="$(arg robot_name)/base_link"/>
+    <child link="$(arg robot_name)/altimeter_link"/>
     <origin xyz="-0.240439 0.067376 -0.35413" rpy="3.1416 0 1.57"/>
   </joint>
   <!-- Thrusters -->
-  <link name="${robot_prefix}left_thruster_link" tf_type="thruster"/>
-  <joint name="${robot_prefix}left_thruster_joint" type="fixed">
-    <parent link="${robot_prefix}base_link"/>
-    <child link="${robot_prefix}left_thruster_link"/>
+  <link name="$(arg robot_name)/left_thruster_link" tf_type="thruster"/>
+  <joint name="$(arg robot_name)/left_thruster_joint" type="fixed">
+    <parent link="$(arg robot_name)/base_link"/>
+    <child link="$(arg robot_name)/left_thruster_link"/>
     <origin xyz="-0.472 -0.28 0.0245" rpy="0.0 0.0 0.0"/>
   </joint>
-  <link name="${robot_prefix}right_thruster_link" tf_type="thruster"/>
-  <joint name="${robot_prefix}right_thruster_joint" type="fixed">
-    <parent link="${robot_prefix}base_link"/>
-    <child link="${robot_prefix}right_thruster_link"/>
+  <link name="$(arg robot_name)/right_thruster_link" tf_type="thruster"/>
+  <joint name="$(arg robot_name)/right_thruster_joint" type="fixed">
+    <parent link="$(arg robot_name)/base_link"/>
+    <child link="$(arg robot_name)/right_thruster_link"/>
     <origin xyz="-0.472 0.28 0.0245" rpy="0.0 0.0 0.0"/>
   </joint>
   <!-- Actuators -->
   <!--
-  <link name="${robot_prefix}status_light_link" tf_type="actuator"/>
-  <joint name="${robot_prefix}status_light_joint" type="fixed">
-    <parent link="${robot_prefix}base_link"/>
-    <child link="${robot_prefix}status_light_link"/>
+  <link name="$(arg robot_name)/status_light_link" tf_type="actuator"/>
+  <joint name="$(arg robot_name)/status_light_joint" type="fixed">
+    <parent link="$(arg robot_name)/base_link"/>
+    <child link="$(arg robot_name)/status_light_link"/>
     <origin xyz="0 0 0" rpy="0 0 0"/>
   </joint>
   -->
   <!-- ROS2 CONTROL -->
-  <ros2_control name="blueboat_thrusters" type="system">
+  <ros2_control name="$(arg robot_name)_thrusters" type="system">
     <hardware>
       <plugin>sura_hardware_interface/ThrustersSystem</plugin>
       <param name="environment">$(arg environment)</param>
     </hardware>
-    <joint name="${robot_prefix}left_thruster_joint">
+    <joint name="$(arg robot_name)/left_thruster_joint">
       <command_interface name="effort"/>
       <state_interface name="effort"/>
-      <param name="lookup_csv">$(arg lookup_csv)</param>
-      <param name="stonefish_topic">$(arg stonefish_topic)</param>
+      <param name="lookup_csv">config/m200_lookup.csv</param>
+      <param name="stonefish_topic">/$(arg robot_name)/controller/thruster_setpoints_sim</param>
       <param name="inverted">false</param>
       <param name="pwm_offset">0.0</param>
       <param name="channel">0</param>
     </joint>
-    <joint name="${robot_prefix}right_thruster_joint">
+    <joint name="$(arg robot_name)/right_thruster_joint">
       <command_interface name="effort"/>
       <state_interface name="effort"/>
-      <param name="lookup_csv">$(arg lookup_csv)</param>
-      <param name="stonefish_topic">$(arg stonefish_topic)</param>
+      <param name="lookup_csv">config/m200_lookup.csv</param>
+      <param name="stonefish_topic">/$(arg robot_name)/controller/thruster_setpoints_sim</param>
       <param name="inverted">true</param>
       <param name="pwm_offset">10.0</param>
@@ -87,5 +83,5 @@
     </joint>
   </ros2_control>
-  <ros2_control name="blueboat_sensors" type="system">
+  <ros2_control name="$(arg robot_name)_sensors" type="system">
     <hardware>
       <plugin>sura_hardware_interface/SensorsSystem</plugin>
@@ -96,6 +92,6 @@
       <param name="broadcaster">imu_broadcaster</param>
       <param name="read_rate_hz">200.0</param>
-      <param name="frame_id">${robot_prefix}imu_link</param>
-      <param name="stonefish_topic">/$(arg robot_namespace)/stonefish/sensors/imu</param>
+      <param name="frame_id">$(arg robot_name)/imu_link</param>
+      <param name="stonefish_topic">/$(arg robot_name)/stonefish/sensors/imu</param>
       <param name="msg_type">sensor_msgs/msg/Imu</param>
       <state_interface name="orientation.x"/>
@@ -114,6 +110,6 @@
       <param name="broadcaster">magnetometer_broadcaster</param>
       <param name="read_rate_hz">50.0</param>
-      <param name="frame_id">${robot_prefix}imu_link</param>
-      <param name="stonefish_topic">/$(arg robot_namespace)/stonefish/sensors/magnetometer</param>
+      <param name="frame_id">$(arg robot_name)/imu_link</param>
+      <param name="stonefish_topic">/$(arg robot_name)/stonefish/sensors/magnetometer</param>
       <param name="msg_type">sensor_msgs/msg/MagneticField</param>
       <state_interface name="magnetic_field.x"/>
@@ -125,5 +121,5 @@
       <param name="broadcaster">battery_broadcaster</param>
       <param name="read_rate_hz">2.0</param>
-      <param name="frame_id">${robot_prefix}base_link</param>
+      <param name="frame_id">$(arg robot_name)/base_link</param>
       <state_interface name="voltage"/>
       <state_interface name="current"/>
@@ -143,5 +139,5 @@
       <param name="scan_length">3000</param>
       <param name="mode_auto">0</param>
-      <param name="frame_id">${robot_prefix}altimeter_link</param>
+      <param name="frame_id">$(arg robot_name)/altimeter_link</param>
       <state_interface name="altitude"/>
       <state_interface name="confidence"/>
@@ -157,6 +153,6 @@
       <param name="gps_serial_port">/dev/ttyAMA5</param>
       <param name="gps_baudrate">230400</param>
-      <param name="frame_id">${robot_prefix}gps_frame</param>
-      <param name="stonefish_topic">/$(arg robot_namespace)/stonefish/sensors/gps</param>
+      <param name="frame_id">$(arg robot_name)/gps_frame</param>
+      <param name="stonefish_topic">/$(arg robot_name)/stonefish/sensors/gps</param>
       <param name="msg_type">sensor_msgs/msg/NavSatFix</param>
       <state_interface name="gps.latitude"/>
@@ -166,5 +162,5 @@
     </sensor>
   </ros2_control>
-  <ros2_control name="blueboat_actuators" type="system">
+  <ros2_control name="$(arg robot_name)_actuators" type="system">
     <hardware>
       <plugin>sura_hardware_interface/ActuatorsSystem</plugin>
@@ -172,5 +168,5 @@
       <param name="status_light_channel">1</param>
     </hardware>
-    <joint name="${robot_prefix}status_light_joint">
+    <joint name="$(arg robot_name)/status_light_joint">
       <param name="interface">sura_hardware_interface/LightBlueboatInterface</param>
       <command_interface name="enabled"/>

File: urdf/blueboat_enu_sim.xacro (robot description, xacro)
@@ -4,5 +4,5 @@
   <xacro:arg name="robot_namespace" default="blueboat"/>
   <xacro:arg name="lookup_csv" default=""/>
-  <xacro:arg name="stonefish_topic" default="/blueboat/catamaran/controller/thruster_setpoints_sim"/>
+  <xacro:arg name="stonefish_topic" default="/blueboat/controller/thruster_setpoints_sim"/>
   <xacro:macro name="blueboat_macro" params="prefix">
     <!-- =========================================================
